File: hardware/blitzbox.brd (EAGLE design)
At the start: 50 x 50 mm, 63 parts, among them IC1 ATMEGA2561-16AU, IC2 TLE8080, IC3 MCP14E10, IC4 FGB3056_F085, IC5 USB6B1, IC6 PL2303SA, IC8 MPXH6400AC6T1, IC9 MPX4250, Q1 ABM3-16.000MHZ-D2Y-T, X2 5566-18

Commit message: Add files via upload
Parts:
- moved C47 3.18 mm to (39.4, 45.7), flipped to the bottom, turned to 0 degrees
- moved C4 0.32 mm to (26.0, 46.4)
Connections:
- new net VUA: IC5.8, IC6.7
- net VU: no longer IC5.8, IC6.7
Routing:
- net VU: track 23.0 -> 7.74 mm, vias 2 -> 1
- net VUA: track 0.00 -> 6.33 mm, vias 0 -> 2
- net +UB: track 9.14 -> 13.0 mm
- net GND: vias 93 -> 94
Changed lines of the file:
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@@
 <element name="R1" library="rcl" package="R0805" value="1k" x="18.415" y="40.3225" rot="R270"/>
 <element name="C3" library="rcl" package="C0805" value="100n" x="23.1775" y="38.735"/>
-<element name="C4" library="rcl" package="C1210" value="22u" x="26.035" y="46.6725" rot="R270"/>
+<element name="C4" library="rcl" package="C1210" value="22u" x="26.035" y="46.355" rot="R270"/>
 <element name="D3" library="st-microelectronics" package="SO08" value="DA112S1" x="34.76625" y="40.64" rot="MR90">
 <attribute name="OC_NEWARK" value="89K0514" x="34.76625" y="40.64" size="1.778" layer="28" rot="MR90" display="off"/>
@@
 <element name="IC6" library="PL2303SA" package="SO-08" value="PL2303SA" x="34.76625" y="34.925" rot="MR90"/>
 <element name="JP3" library="pinhead" package="1X04" value="USB" x="46.99" y="38.4175" rot="R90"/>
-<element name="C47" library="rcl" package="C0805" value="1u" x="42.545" y="45.56125" rot="R90"/>
+<element name="C47" library="rcl" package="C0805" value="1u" x="39.37" y="45.72" rot="MR0"/>
 <element name="L1" library="dp_devices" package="FB805" value="L0805C100MDWIT" x="46.0375" y="44.7675"/>
 <element name="C50" library="rcl" package="C0805" value="1n" x="46.0375" y="46.99" rot="R180"/>
@@
 <wire x1="31.75" y1="47.94" x2="31.59125" y2="47.9425" width="0.2032" layer="1"/>
 <wire x1="31.59125" y1="47.9425" x2="30.63875" y2="46.99" width="0.2032" layer="1"/>
-<wire x1="30.63875" y1="46.99" x2="27.94" y2="46.99" width="0.2032" layer="1"/>
+<wire x1="30.63875" y1="46.99" x2="28.09875" y2="46.99" width="0.2032" layer="1"/>
 <wire x1="21.9075" y1="41.3" x2="22.25" y2="41.3" width="0.2032" layer="1"/>
 <wire x1="22.25" y1="41.3" x2="22.225" y2="41.275" width="0.2032" layer="1"/>
 <wire x1="22.25" y1="41.3" x2="24.13" y2="43.18" width="0.2032" layer="1"/>
-<wire x1="24.13" y1="43.18" x2="24.13" y2="46.19625" width="0.2032" layer="1"/>
-<wire x1="24.13" y1="46.19625" x2="24.60625" y2="46.6725" width="0.2032" layer="1"/>
-<wire x1="24.60625" y1="46.6725" x2="27.6225" y2="46.6725" width="0.2032" layer="1"/>
-<wire x1="27.6225" y1="46.6725" x2="27.94" y2="46.99" width="0.2032" layer="1"/>
+<wire x1="24.13" y1="43.18" x2="24.13" y2="45.87875" width="0.2032" layer="1"/>
+<wire x1="24.13" y1="45.87875" x2="24.60625" y2="46.355" width="0.2032" layer="1"/>
+<wire x1="24.60625" y1="46.355" x2="27.46375" y2="46.355" width="0.2032" layer="1"/>
+<wire x1="27.46375" y1="46.355" x2="28.09875" y2="46.99" width="0.2032" layer="1"/>
 </signal>
 <signal name="GND">
@@
 <via x="19.3675" y="46.355" extent="1-16" drill="0.3048"/>
 <via x="19.3675" y="43.815" extent="1-16" drill="0.3048"/>
-<via x="40.64" y="46.355" extent="1-16" drill="0.3048"/>
+<via x="43.18" y="46.99" extent="1-16" drill="0.3048"/>
 <via x="36.195" y="46.355" extent="1-16" drill="0.3048"/>
 <via x="39.0525" y="18.7325" extent="1-16" drill="0.3048"/>
@@
 <via x="17.145" y="22.86" extent="1-16" drill="0.3048"/>
 <contactref element="IC2" pad="12"/>
+<via x="32.7025" y="1.5875" extent="1-16" drill="0.3048"/>
 </signal>
 <signal name="N$50">
@@
 <wire x1="24.1275" y1="38.735" x2="24.1275" y2="41.59" width="0.4064" layer="1"/>
 <wire x1="24.1275" y1="41.59" x2="26.035" y2="43.4975" width="0.4064" layer="1"/>
-<wire x1="26.035" y1="43.4975" x2="26.035" y2="45.2725" width="0.4064" layer="1"/>
+<wire x1="26.035" y1="43.4975" x2="26.035" y2="44.955" width="0.4064" layer="1"/>
 <wire x1="26.035" y1="43.4975" x2="28.2575" y2="43.4975" width="0.4064" layer="1"/>
 <wire x1="28.2575" y1="43.4975" x2="28.2575" y2="43.7642" width="0.3048" layer="1"/>
@@
 <wire x1="11.97" y1="39.7" x2="11.97" y2="40.3225" width="1.27" layer="1"/>
 <wire x1="12.7" y1="43.7525" x2="11.97" y2="43.7525" width="1.27" layer="1"/>
-<wire x1="11.97" y1="43.7525" x2="11.97" y2="40.3225" width="1.27" layer="1"/>
+<wire x1="11.97" y1="43.7525" x2="11.97" y2="41.8825" width="1.27" layer="1"/>
 <contactref element="X2" pad="1"/>
+<wire x1="11.97" y1="41.8825" x2="11.97" y2="40.3225" width="1.27" layer="1"/>
+<wire x1="8.1475" y1="41.8825" x2="11.97" y2="41.8825" width="1.27" layer="1"/>
 <wire x1="11.59125" y1="39.6875" x2="10.3425" y2="39.6875" width="0.3048" layer="16"/>
 <wire x1="10.3425" y1="39.6875" x2="8.1475" y2="41.8825" width="0.3048" layer="16"/>
-<wire x1="11.59125" y1="39.6875" x2="11.97" y2="39.7" width="0" layer="19" extent="1-16"/>
 </signal>
 <signal name="N$8">
@@
 <contactref element="C47" pad="1"/>
 <contactref element="L1" pad="1"/>
-<contactref element="IC6" pad="7"/>
-<via x="39.37" y="34.925" extent="1-16" drill="0.3048"/>
-<wire x1="37.36625" y1="34.29" x2="38.735" y2="34.29" width="0.3048" layer="16"/>
-<wire x1="38.735" y1="34.29" x2="39.37" y2="34.925" width="0.3048" layer="16"/>
-<wire x1="39.37" y1="34.925" x2="39.37" y2="38.89375" width="0.3048" layer="1"/>
-<wire x1="39.37" y1="38.89375" x2="40.3225" y2="39.84625" width="0.3048" layer="1"/>
-<wire x1="40.3225" y1="39.84625" x2="40.3225" y2="42.38625" width="0.3048" layer="1"/>
-<wire x1="40.3225" y1="42.38625" x2="42.545" y2="44.60875" width="0.3048" layer="1"/>
-<wire x1="42.545" y1="44.61125" x2="42.545" y2="44.60875" width="0.3048" layer="1"/>
-<wire x1="45.1875" y1="44.7675" x2="42.70125" y2="44.7675" width="0.3048" layer="1"/>
-<wire x1="42.70125" y1="44.7675" x2="42.545" y2="44.61125" width="0.3048" layer="1"/>
 <contactref element="IC5" pad="1"/>
-<contactref element="IC5" pad="8"/>
-<via x="40.3225" y="39.84625" extent="1-16" drill="0.3048"/>
-<wire x1="40.3225" y1="38.04" x2="40.3225" y2="39.84625" width="0.3048" layer="16"/>
-<wire x1="40.3225" y1="43.24" x2="40.3225" y2="38.04" width="0.3048" layer="16"/>
+<via x="42.545" y="45.72" extent="1-16" drill="0.3048"/>
+<wire x1="40.3225" y1="43.24" x2="40.32" y2="43.24" width="0.3048" layer="16"/>
+<wire x1="40.32" y1="43.24" x2="40.32" y2="45.72" width="0.3048" layer="16"/>
+<wire x1="45.1875" y1="44.7675" x2="43.4975" y2="44.7675" width="0.3048" layer="1"/>
+<wire x1="43.4975" y1="44.7675" x2="42.545" y2="45.72" width="0.3048" layer="1"/>
+<wire x1="40.32" y1="45.72" x2="42.545" y2="45.72" width="0.3048" layer="16"/>
 </signal>
 <signal name="+5VU">
@@
 <wire x1="26.285" y1="9.2075" x2="26.19375" y2="9.2075" width="0.2032" layer="1"/>
 </signal>
+<signal name="VUA">
+<contactref element="IC5" pad="8"/>
+<contactref element="IC6" pad="7"/>
+<via x="39.37" y="34.925" extent="1-16" drill="0.3048"/>
+<via x="39.37" y="37.62375" extent="1-16" drill="0.3048"/>
+<wire x1="40.3225" y1="38.04" x2="40.3225" y2="37.62375" width="0.3048" layer="16"/>
+<wire x1="40.3225" y1="37.62375" x2="39.37" y2="37.62375" width="0.3048" layer="16"/>
+<wire x1="37.36625" y1="34.29" x2="38.735" y2="34.29" width="0.3048" layer="16"/>
+<wire x1="38.735" y1="34.29" x2="39.37" y2="34.925" width="0.3048" layer="16"/>
+<wire x1="39.37" y1="34.925" x2="39.37" y2="37.62375" width="0.3048" layer="1"/>
+</signal>
 </signals>
