File: hardware/blitzbox.sch (EAGLE design)
At the start: 63 parts, among them IC1 ATMEGA2561-16AU, IC2 TLE8080, IC3 MCP14E10, IC4 FGB3056_F085, IC5 USB6B1, IC6 PL2303SA, IC8 MPXH6400AC6T1, IC9 MPX4250, Q1 ABM3-16.000MHZ-D2Y-T, X2 5566-18

Commit message: Add files via upload
Connections:
- new net VUA: IC5.VCC@2, IC6.VBUS
- net VU: no longer IC5.VCC@2, IC6.VBUS
Changed lines of the file:
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@@
-</segment>
-<segment>
-<pinref part="IC6" gate="G$1" pin="VBUS"/>
-<wire x1="208.28" y1="38.1" x2="203.2" y2="38.1" width="0.1524" layer="91"/>
-<label x="203.2" y="38.1" size="1.778" layer="95"/>
 </segment>
 <segment>
@@
 <wire x1="231.14" y1="81.28" x2="226.06" y2="81.28" width="0.1524" layer="91"/>
 <label x="226.06" y="81.28" size="1.778" layer="95"/>
-</segment>
-<segment>
-<pinref part="IC5" gate="G$1" pin="VCC@2"/>
-<wire x1="246.38" y1="81.28" x2="251.46" y2="81.28" width="0.1524" layer="91"/>
-<label x="248.92" y="81.28" size="1.778" layer="95"/>
 </segment>
 </net>
@@
 </segment>
 </net>
+<net name="VUA" class="0">
+<segment>
+<pinref part="IC5" gate="G$1" pin="VCC@2"/>
+<wire x1="246.38" y1="81.28" x2="251.46" y2="81.28" width="0.1524" layer="91"/>
+<label x="248.92" y="81.28" size="1.778" layer="95"/>
+</segment>
+<segment>
+<pinref part="IC6" gate="G$1" pin="VBUS"/>
+<wire x1="208.28" y1="38.1" x2="203.2" y2="38.1" width="0.1524" layer="91"/>
+<label x="203.2" y="38.1" size="1.778" layer="95"/>
+</segment>
+</net>
